File: OHAK_130.sch (KiCad schematic (older format))
At the start: 42 parts, among them P1 CONN_01X10, P2 USB_OTG, Q1 Q_NMOS_GSD, Q2 Q_NMOS_GSD, U1 rfd_77101, U2 MAX30100, U3 NCP551, U4 BMI160, U5 MCP73831, U6 NCP551

Commit message: updated shematic and library
Parts:
- removed Q1, Q2: Q_NMOS_GSD, TO_SOT_Packages_SMD:SOT-23, symbol Device:Q_NMOS_GSD
- removed R10, R11, R16, R9: 10K, Capacitors_SMD:C_0603, symbol Device:R
- removed U3, U6: NCP551, TO_SOT_Packages_SMD:SOT-23-5, symbol Solutions:NCP551
- added C15, C16: 0.1uF, Capacitors_SMD:C_0402, symbol Device:C
- added U3, U6: MIC5365-X.XYMT-TZ, Solutions:MLF-4 1mm x 1mm, symbol Solutions:MIC5365-X.XYMT-TZ
- added U7: TXS0102_LEVEL_SHIFTER_X2SON8, Solutions:X2SON8_1.4mm_x_1mm, symbol Solutions:TXS0102_LEVEL_SHIFTER_X2SON8
- added U8: MAX809, TO_SOT_Packages_SMD:SOT-323_SC-70, symbol Solutions:MAX809
- C1, C10, C11, C12, C13, C14, C2, C3, C4, C5, C6, C7, C8, C9, R1, R12, R13, R14, R15, R17, R2, R5, R7, R8: footprint Capacitors_SMD:C_0603 -> Capacitors_SMD:C_0402
Connections:
- net +1V8: now also C15.2, U3.1 (VOUT), U7.1 (VccA), U7.5 (OE)
- net 1V8_SCL: now also U7.3 (A2)
- net 1V8_SDA: now also U7.2 (A1)
- net 3V3_SCL: now also U7.6 (B2)
- net 3V3_SDA: now also U7.7 (B1)
- net GND: now also C15.1, C16.1, U3.2 (GND), U3.5 (EP), U6.2 (GND), U6.5 (EP), U7.4 (GND), U8.1 (GND)
- net VDD: now also C16.2, U6.1 (VOUT), U7.8 (VccB)
- net VPP: now also U3.4 (VIN), U6.4 (VIN), U8.3 (VDD)
- new net EN: U3.3 (EN), U6.3 (EN), U8.2 (RST)
Other:
- note added: "MAX809SQ308T1G"
- note added: "MIC5365-1.8YMT-TZ"
- note added: "MIC5365-3.0YMT-TZ"
- note removed: "12V MAX INPUT"
- note removed: "ADP162AUJZ-1.8-R7"
- note removed: "ADP162AUJZ-3.3-R7"
- moved on the sheet: C13, C14, C9, R7, R8, U4

Commit message: moved parts to top layer and routed board
Parts:
- P1: value CONN_01X10 -> CONN_01X08; footprint Solutions:4u-0201GDVE06 -> Solutions:M50-3140845_1x8_SMT_F; symbol Connector:Conn_01x10_Female -> Connector_Generic:Conn_01x08
Connections:
- net BMI_INT1: now also U1.40 (P0.29); no longer U1.33 (P0.20)
- net BMI_INT2: now also U1.39 (P0.28); no longer U1.35 (P0.24)
- net B_LED: now also U1.33 (P0.20); no longer U1.38 (P0.25)
- net EN: no longer U3.3 (EN)
- net GND: no longer P1.10 (Pin_10), P1.9 (Pin_9)
- net G_LED: now also U1.34 (P0.23); no longer U1.40 (P0.29)
- net R_LED: now also U1.35 (P0.24); no longer U1.39 (P0.28)
- net VDD: now also C8.2, U3.3 (EN), U3.4 (VIN)
- net VPP: no longer C8.2, U3.4 (VIN)
- net PIN_4: no longer names the net of U1.32 (P0.04/AIN5)
- net PIN_4: no longer P1.6 (Pin_6)
- new net PIN_25: P1.6 (Pin_6), U1.38 (P0.25)
Other:
- moved on the sheet: C10, C12, C13, C8, C9, U3, U6
Changed lines of the file:
@@
 EESchema Schematic File Version 4
-LIBS:OHAK_130-cache
 EELAYER 26 0
 EELAYER END
@@
 	1    0    0    -1
 $EndComp
-Text Label 6500 6200 1    60   ~ 0
+Text Label 6750 5950 2    60   ~ 0
 SIM_RX
-Text Label 6700 6200 1    60   ~ 0
+Text Label 6750 5750 2    60   ~ 0
 SIM_TX
-Text Label 6900 5700 0    60   ~ 0
+Text Label 6100 5550 2    60   ~ 0
 SIM_RST
 Text Label 3550 6500 3    60   ~ 0
@@
 L power:VDD #PWR06
 U 1 1 57CDC75F
-P 7500 1950
-F 0 "#PWR06" H 7500 1800 50  0001 C CNN
-F 1 "VDD" H 7500 2100 50  0000 C CNN
-F 2 "" H 7500 1950 50  0000 C CNN
-F 3 "" H 7500 1950 50  0000 C CNN
-	1    7500 1950
+P 7350 1050
+F 0 "#PWR06" H 7350 900 50  0001 C CNN
+F 1 "VDD" H 7350 1200 50  0000 C CNN
+F 2 "" H 7350 1050 50  0000 C CNN
+F 3 "" H 7350 1050 50  0000 C CNN
+	1    7350 1050
 	1    0    0    -1
 $EndComp
@@
 L Device:C C8
 U 1 1 57CDCC34
-P 5750 1350
-F 0 "C8" H 5775 1450 50  0000 L CNN
-F 1 "1uF" H 5775 1250 50  0000 L CNN
-F 2 "Capacitors_SMD:C_0402" H 5788 1200 50  0001 C CNN
-F 3 "" H 5750 1350 50  0000 C CNN
-	1    5750 1350
+P 5750 2250
+F 0 "C8" H 5775 2350 50  0000 L CNN
+F 1 "1uF" H 5775 2150 50  0000 L CNN
+F 2 "Capacitors_SMD:C_0402" H 5788 2100 50  0001 C CNN
+F 3 "" H 5750 2250 50  0000 C CNN
+	1    5750 2250
 	-1   0    0    1
 $EndComp
@@
 L Device:C C9
 U 1 1 57CDCEC9
-P 7500 1350
-F 0 "C9" H 7525 1450 50  0000 L CNN
-F 1 "1uF" H 7525 1250 50  0000 L CNN
-F 2 "Capacitors_SMD:C_0402" H 7538 1200 50  0001 C CNN
-F 3 "" H 7500 1350 50  0000 C CNN
-	1    7500 1350
+P 7500 2250
+F 0 "C9" H 7525 2350 50  0000 L CNN
+F 1 "1uF" H 7525 2150 50  0000 L CNN
+F 2 "Capacitors_SMD:C_0402" H 7538 2100 50  0001 C CNN
+F 3 "" H 7500 2250 50  0000 C CNN
+	1    7500 2250
 	-1   0    0    1
 $EndComp
 Text Label 4900 3950 0    60   ~ 0
 MAX_INT
-Text Label 4900 4150 0    60   ~ 0
+Text Label 4900 4550 0    60   ~ 0
 R_LED
 Text Notes 3750 900  0    60   ~ 0
@@
 L power:GND #PWR08
 U 1 1 580BABD6
-P 5850 6000
-F 0 "#PWR08" H 5850 5750 50  0001 C CNN
-F 1 "GND" H 5850 5850 50  0000 C CNN
-F 2 "" H 5850 6000 50  0000 C CNN
-F 3 "" H 5850 6000 50  0000 C CNN
-	1    5850 6000
+P 6250 6350
+F 0 "#PWR08" H 6250 6100 50  0001 C CNN
+F 1 "GND" H 6250 6200 50  0000 C CNN
+F 2 "" H 6250 6350 50  0000 C CNN
+F 3 "" H 6250 6350 50  0000 C CNN
+	1    6250 6350
 	1    0    0    -1
 $EndComp
@@
 L Device:C C10
 U 1 1 580BBC08
-P 6900 5850
-F 0 "C10" H 6700 5950 50  0000 L CNN
-F 1 "0.1uF" H 6650 5750 50  0000 L CNN
-F 2 "Capacitors_SMD:C_0402" H 6938 5700 50  0001 C CNN
-F 3 "" H 6900 5850 50  0000 C CNN
-	1    6900 5850
-	-1   0    0    -1
+P 6400 5550
+F 0 "C10" V 6350 5600 50  0000 L CNN
+F 1 "0.1uF" V 6350 5300 50  0000 L CNN
+F 2 "Capacitors_SMD:C_0402" H 6438 5400 50  0001 C CNN
+F 3 "" H 6400 5550 50  0000 C CNN
+	1    6400 5550
+	0    -1   1    0
 $EndComp
 $Comp
@@
 	1    0    0    -1
 $EndComp
+Text Label 4900 4050 0    60   ~ 0
+BMI_INT1
+Text Label 4900 4150 0    60   ~ 0
+BMI_INT2
 Text Label 4900 4750 0    60   ~ 0
-BMI_INT1
-Text Label 4900 4550 0    60   ~ 0
-BMI_INT2
-Text Label 4900 4250 0    60   ~ 0
 B_LED
-Text Label 4900 4050 0    60   ~ 0
+Text Label 4900 4650 0    60   ~ 0
 G_LED
 $Comp
@@
 L Device:C C12
 U 1 1 588CF248
-P 5750 2250
-F 0 "C12" H 5775 2350 50  0000 L CNN
-F 1 "1uF" H 5775 2150 50  0000 L CNN
-F 2 "Capacitors_SMD:C_0402" H 5788 2100 50  0001 C CNN
-F 3 "" H 5750 2250 50  0000 C CNN
-	1    5750 2250
+P 5750 1350
+F 0 "C12" H 5775 1450 50  0000 L CNN
+F 1 "1uF" H 5775 1250 50  0000 L CNN
+F 2 "Capacitors_SMD:C_0402" H 5788 1200 50  0001 C CNN
+F 3 "" H 5750 1350 50  0000 C CNN
+	1    5750 1350
 	-1   0    0    1
 $EndComp
@@
 L Device:C C13
 U 1 1 588CF2DB
-P 7500 2250
-F 0 "C13" H 7525 2350 50  0000 L CNN
-F 1 "1uF" H 7525 2150 50  0000 L CNN
-F 2 "Capacitors_SMD:C_0402" H 7538 2100 50  0001 C CNN
-F 3 "" H 7500 2250 50  0000 C CNN
-	1    7500 2250
+P 7500 1350
+F 0 "C13" H 7525 1450 50  0000 L CNN
+F 1 "1uF" H 7525 1250 50  0000 L CNN
+F 2 "Capacitors_SMD:C_0402" H 7538 1200 50  0001 C CNN
+F 3 "" H 7500 1350 50  0000 C CNN
+	1    7500 1350
 	-1   0    0    1
 $EndComp
@@
 	5600 1150 5600 1050
 Wire Wire Line
-	6200 5900 6200 6200
-Wire Wire Line
-	6900 6200 6900 6000
+	6750 5550 6550 5550
 Wire Wire Line
 	5050 1500 5050 1550
@@
 Wire Wire Line
 	2500 9500 2800 9500
-Wire Wire Line
-	6300 5700 6300 6200
 Wire Wire Line
 	1350 1150 2250 1150
@@
 Wire Wire Line
 	2050 1350 2050 1400
-$Comp
-L power:VPP #PWR017
-U 1 1 588CF7C8
-P 5600 2000
-F 0 "#PWR017" H 5600 1850 50  0001 C CNN
-F 1 "VPP" H 5600 2150 50  0000 C CNN
-F 2 "" H 5600 2000 50  0000 C CNN
-F 3 "" H 5600 2000 50  0000 C CNN
-	1    5600 2000
-	1    0    0    -1
-$EndComp
 Wire Wire Line
 	5600 2050 5750 2050
@@
 L power:+1V8 #PWR019
 U 1 1 588D052F
-P 7350 1050
-F 0 "#PWR019" H 7350 900 50  0001 C CNN
-F 1 "+1V8" H 7350 1190 50  0000 C CNN
-F 2 "" H 7350 1050 50  0000 C CNN
-F 3 "" H 7350 1050 50  0000 C CNN
-	1    7350 1050
+P 7500 1950
+F 0 "#PWR019" H 7500 1800 50  0001 C CNN
+F 1 "+1V8" H 7500 2090 50  0000 C CNN
+F 2 "" H 7500 1950 50  0000 C CNN
+F 3 "" H 7500 1950 50  0000 C CNN
+	1    7500 1950
 	1    0    0    -1
 $EndComp
@@
 L power:VDD #PWR023
 U 1 1 588D97A7
-P 6300 5700
-F 0 "#PWR023" H 6300 5550 50  0001 C CNN
-F 1 "VDD" H 6300 5850 50  0000 C CNN
-F 2 "" H 6300 5700 50  0000 C CNN
-F 3 "" H 6300 5700 50  0000 C CNN
-	1    6300 5700
-	1    0    0    -1
-$EndComp
-$Comp
-L Connector:Conn_01x10_Female P1
+P 6250 6050
+F 0 "#PWR023" H 6250 5900 50  0001 C CNN
+F 1 "VDD" H 6250 6200 50  0000 C CNN
+F 2 "" H 6250 6050 50  0000 C CNN
+F 3 "" H 6250 6050 50  0000 C CNN
+	1    6250 6050
+	1    0    0    -1
+$EndComp
+$Comp
+L Connector_Generic:Conn_01x08 P1
 U 1 1 588D9B00
-P 6500 6400
-F 0 "P1" H 6500 6950 50  0000 C CNN
-F 1 "CONN_01X10" V 6600 6400 50  0000 C CNN
-F 2 "Solutions:4u-0201GDVE06" H 6500 6400 50  0001 C CNN
-F 3 "" H 6500 6400 50  0000 C CNN
-	1    6500 6400
-	0    1    1    0
-$EndComp
-Wire Wire Line
-	6100 5900 6100 6200
-Wire Wire Line
-	5850 5900 6000 5900
-Connection ~ 6000 5900
-Wire Wire Line
-	6000 5900 6000 6200
-Connection ~ 6100 5900
-Wire Wire Line
-	5850 6000 5850 5900
+P 6950 5850
+F 0 "P1" H 6950 6250 50  0000 C CNN
+F 1 "CONN_01X08" V 7050 5850 50  0000 C CNN
+F 2 "Solutions:M50-3140845_1x8_SMT_F" H 6950 5850 50  0001 C CNN
+F 3 "" H 6950 5850 50  0000 C CNN
+	1    6950 5850
+	1    0    0    -1
+$EndComp
 Text Label 3050 6500 3    60   ~ 0
 PIN_3
 Text Label 3250 6500 3    60   ~ 0
 PIN_2
-Text Label 4900 4850 0    60   ~ 0
-PIN_4
-Text Label 6400 6200 1    60   ~ 0
-PIN_4
-Text Label 6600 6200 1    60   ~ 0
+Text Label 4900 4250 0    60   ~ 0
+PIN_25
+Text Label 6750 6050 2    60   ~ 0
+PIN_25
+Text Label 6750 5850 2    60   ~ 0
 PIN_2
-Text Label 6800 6200 1    60   ~ 0
+Text Label 6750 5650 2    60   ~ 0
 PIN_3
 Text Label 2950 6500 3    60   ~ 0
@@
 Wire Wire Line
 	2050 2200 4050 2200
-Wire Wire Line
-	6000 5900 6100 5900
-Wire Wire Line
-	6100 5900 6200 5900
 Wire Wire Line
 	1050 1750 1450 1750
@@
 L Solutions:MIC5365-X.XYMT-TZ U3
 U 1 1 5C5A898A
+P 6600 2050
+F 0 "U3" H 6450 2150 60  0000 C CNN
+F 1 "MIC5365-X.XYMT-TZ" H 6550 1750 60  0000 C CNN
+F 2 "Solutions:MLF-4 1mm x 1mm" H 6600 2050 60  0001 C CNN
+F 3 "" H 6600 2050 60  0001 C CNN
+	1    6600 2050
+	1    0    0    -1
+$EndComp
+$Comp
+L Solutions:MIC5365-X.XYMT-TZ U6
+U 1 1 5C5A8CE1
 P 6600 1150
-F 0 "U3" H 6450 1250 60  0000 C CNN
-F 1 "MIC5365-X.XYMT-TZ" H 6550 850 60  0000 C CNN
+F 0 "U6" H 6450 1250 60  0000 C CNN
+F 1 "MIC5365-X.XYMT-TZ" H 6600 850 60  0000 C CNN
 F 2 "Solutions:MLF-4 1mm x 1mm" H 6600 1150 60  0001 C CNN
 F 3 "" H 6600 1150 60  0001 C CNN
 	1    6600 1150
-	1    0    0    -1
-$EndComp
-$Comp
-L Solutions:MIC5365-X.XYMT-TZ U6
-U 1 1 5C5A8CE1
-P 6600 2050
-F 0 "U6" H 6450 2150 60  0000 C CNN
-F 1 "MIC5365-X.XYMT-TZ" H 6600 1750 60  0000 C CNN
-F 2 "Solutions:MLF-4 1mm x 1mm" H 6600 2050 60  0001 C CNN
-F 3 "" H 6600 2050 60  0001 C CNN
-	1    6600 2050
 	1    0    0    -1
 $EndComp
@@
 	5750 1150 6200 1150
 Wire Wire Line
-	5750 2050 6200 2050
+	5750 2050 6050 2050
 Wire Wire Line
 	7050 2050 7500 2050
@@
 	7200 2550 7200 2450
 Text Label 6200 1250 2    60   ~ 0
-EN
-Text Label 6200 2150 2    60   ~ 0
 EN
 $Comp
@@
 Text Label 7000 3350 0    60   ~ 0
 EN
+Text Notes 6100 1900 0    60   ~ 0
+MIC5365-1.8YMT-TZ
 Text Notes 6100 1000 0    60   ~ 0
-MIC5365-1.8YMT-TZ
-Text Notes 5900 1900 0    60   ~ 0
 MIC5365-3.0YMT-TZ
 Text Notes 6350 3100 0    60   ~ 0
 MAX809SQ308T1G
+Wire Wire Line
+	6250 5550 6100 5550
+Wire Wire Line
+	6750 6150 6250 6150
+Wire Wire Line
+	6250 6150 6250 6050
+Wire Wire Line
+	6750 6250 6250 6250
+Wire Wire Line
+	6250 6250 6250 6350
+$Comp
+L power:VDD #PWR0101
+U 1 1 5C75E84A
+P 5600 2000
+F 0 "#PWR0101" H 5600 1850 50  0001 C CNN
+F 1 "VDD" H 5600 2150 50  0000 C CNN
+F 2 "" H 5600 2000 50  0000 C CNN
+F 3 "" H 5600 2000 50  0000 C CNN
+	1    5600 2000
+	1    0    0    -1
+$EndComp
+Wire Wire Line
+	6200 2150 6050 2150
+Wire Wire Line
+	6050 2150 6050 2050
+Connection ~ 6050 2050
+Wire Wire Line
+	6050 2050 6200 2050
 $EndSCHEMATC

Commit message: finished BOM
Parts:
- R12, R17: value 30R -> 100R
- R5: value 130R -> 100R
Changed lines of the file:
@@
 P 1250 5450
 F 0 "R5" V 1330 5450 50  0000 C CNN
-F 1 "130R" V 1250 5450 50  0000 C CNN
+F 1 "100R" V 1250 5450 50  0000 C CNN
 F 2 "Capacitors_SMD:C_0402" V 1180 5450 50  0001 C CNN
 F 3 "" H 1250 5450 50  0000 C CNN
@@
 P 1050 5450
 F 0 "R12" V 1130 5450 50  0000 C CNN
-F 1 "30R" V 1050 5450 50  0000 C CNN
+F 1 "100R" V 1050 5450 50  0000 C CNN
 F 2 "Capacitors_SMD:C_0402" V 980 5450 50  0001 C CNN
 F 3 "" H 1050 5450 50  0000 C CNN
@@
 P 850 5450
 F 0 "R17" V 930 5450 50  0000 C CNN
-F 1 "30R" V 850 5450 50  0000 C CNN
+F 1 "100R" V 850 5450 50  0000 C CNN
 F 2 "Capacitors_SMD:C_0402" V 780 5450 50  0001 C CNN
 F 3 "" H 850 5450 50  0000 C CNN

Commit message: fixed mis pinned part. moved stuff around
Parts:
- D1: value Led_RGB_CA -> ASMB-KTF0-0A306
- D3: value Dialight_R_G_LED -> 18-225SURSYGC/S530-A4/E4/TR8
- P1: value CONN_01X08 -> M50-3140845
- U3: value MIC5365-X.XYMT-TZ -> MIC5365-1.8YMT-TZ
- U5: value MCP73831 -> MCP73831T-2ATI/OT
- U6: value MIC5365-X.XYMT-TZ -> MIC5365-3.0YMT-TZ
- U7: value TXS0102_LEVEL_SHIFTER_X2SON8 -> TXS0102DQER
- U8: value MAX809 -> MAX809SQ308T1G
Other:
- note added: "ALT: CLMVB-FKA-\nCFHEHLCBB7a363"
- note added: "GPIO 3 / ANALOG 4\nGPIO 1 / ANALOG 2\nGPIO 2 / ANALOG 3\nGPIO 0 / AREF 0\nGPIO 25\n"
- note removed: "2N7002ET1G\n"
- note removed: "CLMVB-FKA-\nCFHEHLCBB7a363"
- note removed: "MAX809SQ308T1G"
- note removed: "MIC5365-1.8YMT-TZ"
- note removed: "MIC5365-3.0YMT-TZ"
- moved on the sheet: D3
Changed lines of the file:
@@
 EESchema Schematic File Version 4
+LIBS:OHAK_130-cache
 EELAYER 26 0
 EELAYER END
@@
 Text Label 2800 9400 0    60   ~ 0
 3V3_SCL
-Text Notes 5050 8800 0    60   ~ 0
-2N7002ET1G\n
 $Comp
 L power:VDD #PWR013
@@
 L Solutions:Dialight_R_G_LED D3
 U 1 1 5820CD7B
-P 2150 1700
-F 0 "D3" H 2150 1925 50  0000 C CNN
-F 1 "Dialight_R_G_LED" H 2150 2050 50  0000 C CNN
-F 2 "Solutions:0606_Bi-Color" H 2150 1700 50  0001 C CNN
-F 3 "" H 2150 1700 50  0000 C CNN
-	1    2150 1700
+P 2000 1700
+F 0 "D3" H 2000 1925 50  0000 C CNN
+F 1 "18-225SURSYGC/S530-A4/E4/TR8" V 2600 1600 50  0000 C CNN
+F 2 "Solutions:0606_Bi-Color" H 2000 1700 50  0001 C CNN
+F 3 "" H 2000 1700 50  0000 C CNN
+	1    2000 1700
 	0    -1   -1   0
 $EndComp
@@
 P 3450 1300
 F 0 "U5" H 3250 1550 60  0000 C CNN
-F 1 "MCP73831" H 3450 1050 60  0000 C CNN
+F 1 "MCP73831T-2ATI/OT" H 3450 1050 60  0000 C CNN
 F 2 "TO_SOT_Packages_SMD:SOT-23-5" H 3800 1550 60  0001 C CNN
 F 3 "" H 3800 1550 60  0000 C CNN
@@
 	2500 9500 2800 9500
 Wire Wire Line
-	1350 1150 2250 1150
-Wire Wire Line
-	2250 2100 2800 2100
+	1350 1150 2100 1150
+Wire Wire Line
+	2100 2100 2800 2100
 Wire Wire Line
 	2800 2100 2800 1900
@@
 Connection ~ 2800 1450
 Wire Wire Line
-	2250 1150 2250 1400
-Connection ~ 2250 1150
+	2100 1150 2100 1400
+Connection ~ 2100 1150
 Wire Wire Line
 	950  1750 950  1900
@@
 Connection ~ 950  1900
 Wire Wire Line
-	1450 2200 2050 2200
+	1450 2200 1900 2200
 Wire Wire Line
 	3950 1300 4200 1300
@@
 	4950 8900 6050 8900
 Wire Wire Line
-	2250 2000 2250 2100
-Wire Wire Line
-	2050 2000 2050 2200
-Connection ~ 2050 2200
-Wire Wire Line
-	2400 1350 2050 1350
-Wire Wire Line
-	2050 1350 2050 1400
+	2100 2000 2100 2100
+Wire Wire Line
+	1900 2000 1900 2200
+Connection ~ 1900 2200
 Wire Wire Line
 	5600 2050 5750 2050
@@
 P 1050 5050
 F 0 "D1" H 1050 5400 50  0000 C CNN
-F 1 "Led_RGB_CA" V 1250 5300 50  0000 C CNN
+F 1 "ASMB-KTF0-0A306" V 50  5100 50  0000 C CNN
 F 2 "Solutions:CLMVB-FKA-CFHEHLCBB7a363" H 1005 5000 50  0001 C CNN
 F 3 "" H 1005 5000 50  0000 C CNN
@@
 Wire Wire Line
 	1050 4850 1050 4700
-Text Notes 550  6150 0    60   ~ 0
-CLMVB-FKA-\nCFHEHLCBB7a363
+Text Notes 600  6300 0    60   ~ 0
+ALT: CLMVB-FKA-\nCFHEHLCBB7a363
 $Comp
 L power:VDD #PWR023
@@
 P 6950 5850
 F 0 "P1" H 6950 6250 50  0000 C CNN
-F 1 "CONN_01X08" V 7050 5850 50  0000 C CNN
+F 1 "M50-3140845" H 6750 5350 50  0000 C CNN
 F 2 "Solutions:M50-3140845_1x8_SMT_F" H 6950 5850 50  0001 C CNN
 F 3 "" H 6950 5850 50  0000 C CNN
@@
 	2800 1450 2800 1600
 Wire Wire Line
-	2250 1150 2950 1150
+	2100 1150 2950 1150
 Wire Wire Line
 	1450 1900 1450 2200
@@
 	6250 4850 6300 4850
 Wire Wire Line
-	2050 2200 4050 2200
+	1900 2200 4050 2200
 Wire Wire Line
 	1050 1750 1450 1750
@@
 P 2200 7650
 F 0 "U7" H 1950 7900 60  0000 C CNN
-F 1 "TXS0102_LEVEL_SHIFTER_X2SON8" H 2100 7350 60  0000 C CNN
+F 1 "TXS0102DQER" H 2200 7350 60  0000 C CNN
 F 2 "Solutions:X2SON8_1.4mm_x_1mm" H 2050 7800 60  0001 C CNN
 F 3 "" H 2050 7800 60  0001 C CNN
@@
 P 6600 2050
 F 0 "U3" H 6450 2150 60  0000 C CNN
-F 1 "MIC5365-X.XYMT-TZ" H 6550 1750 60  0000 C CNN
+F 1 "MIC5365-1.8YMT-TZ" H 6550 1750 60  0000 C CNN
 F 2 "Solutions:MLF-4 1mm x 1mm" H 6600 2050 60  0001 C CNN
 F 3 "" H 6600 2050 60  0001 C CNN
@@
 P 6600 1150
 F 0 "U6" H 6450 1250 60  0000 C CNN
-F 1 "MIC5365-X.XYMT-TZ" H 6600 850 60  0000 C CNN
+F 1 "MIC5365-3.0YMT-TZ" H 6600 850 60  0000 C CNN
 F 2 "Solutions:MLF-4 1mm x 1mm" H 6600 1150 60  0001 C CNN
 F 3 "" H 6600 1150 60  0001 C CNN
@@
 P 6600 3350
 F 0 "U8" H 6500 3550 60  0000 C CNN
-F 1 "MAX809" H 6600 3150 60  0000 C CNN
+F 1 "MAX809SQ308T1G" H 6750 3150 60  0000 C CNN
 F 2 "TO_SOT_Packages_SMD:SOT-323_SC-70" H 6600 3350 60  0001 C CNN
 F 3 "" H 6600 3350 60  0001 C CNN
@@
 Text Label 7000 3350 0    60   ~ 0
 EN
-Text Notes 6100 1900 0    60   ~ 0
-MIC5365-1.8YMT-TZ
-Text Notes 6100 1000 0    60   ~ 0
-MIC5365-3.0YMT-TZ
-Text Notes 6350 3100 0    60   ~ 0
-MAX809SQ308T1G
 Wire Wire Line
 	6250 5550 6100 5550
@@
 Wire Wire Line
 	6050 2050 6200 2050
+Text Notes 7050 6050 0    60   ~ 0
+GPIO 3 / ANALOG 4\nGPIO 1 / ANALOG 2\nGPIO 2 / ANALOG 3\nGPIO 0 / AREF 0\nGPIO 25\n
+Wire Wire Line
+	1900 1350 1900 1400
+Wire Wire Line
+	1900 1350 2400 1350
 $EndSCHEMATC

Commit message: minor changes
Parts:
- R2: value 10K -> 4K7
Other:
- note added: "Change pullup connection to VDD"
- note added: "center this LED\non the board"
Changed lines of the file:
@@
 P 6650 7500
 F 0 "R2" V 6730 7500 50  0000 C CNN
-F 1 "10K" V 6650 7500 50  0000 C CNN
+F 1 "4K7" V 6650 7500 50  0000 C CNN
 F 2 "Capacitors_SMD:C_0402" V 6580 7500 50  0001 C CNN
 F 3 "" H 6650 7500 50  0000 C CNN
@@
 Wire Wire Line
 	1900 1350 2400 1350
+Text Notes 6050 7250 0    60   ~ 0
+Change pullup connection to VDD
+Text Notes 700  4450 0    60   ~ 0
+center this LED\non the board
 $EndSCHEMATC
